File: Board Files/Mainboard.brd (EAGLE design)
At the start: 268 x 101.6 mm, 119 parts, among them J1 I2C Display

Commit message: Cleaned up more routing
-Still need to do physical layout check
Parts:
- moved R54 1.27 mm to (153.7, 87.0)
- moved R53 0.63 mm to (143.5, 87.0)
Routing:
- net SWITCH2-3: track 119.6 -> 143.7 mm, vias 1 -> 3
- net SWITCH1-6: track 121.1 -> 143.0 mm
- net SWITCH1-4: track 146.7 -> 165.9 mm
- net SWITCH3-3: track 118.6 -> 108.6 mm, vias 3 -> 5
- net SWITCH2-1: track 151.3 -> 159.5 mm, vias 1 -> 3
- net LED1-7: track 111.9 -> 119.7 mm, vias 3 -> 5
- net SWITCH1-2: track 192.1 -> 199.7 mm
- net LED3-6: track 56.6 -> 62.5 mm
- net SWITCH2-5: track 115.2 -> 120.3 mm, vias 2 -> 6
- net SWITCH2-2: track 166.4 -> 171.2 mm
- net LED1-8: track 95.7 -> 99.0 mm
- net LED1-5: track 137.7 -> 139.6 mm
- net SWITCH2-6: track 90.9 -> 89.5 mm
- net LED2-2: track 101.1 -> 102.6 mm
- net N$25: track 8.58 -> 9.85 mm
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
Commit message: Finished Mainboard V1.0
-Added holes
-Labeled everything
-Final trace cleanup
Parts:
- S5: value CHERRY_LED -> (none)
- moved D22 19.9 mm to (238.8, 29.8)
- moved R43 19.9 mm to (238.8, 34.3)
- moved R44 19.9 mm to (238.8, 9.53)
- moved S22 19.9 mm to (238.8, 19.1)
- moved D12 19.9 mm to (124.5, 29.8)
- moved R23 19.9 mm to (124.5, 34.3)
- moved R24 19.9 mm to (124.5, 9.53)
- moved S12 19.9 mm to (124.5, 19.1)
- moved D2 19.9 mm to (19.7, 64.1)
- moved D11 19.9 mm to (114.9, 64.1)
- moved D14 19.9 mm to (153.0, 64.1)
- moved D16 19.9 mm to (172.1, 64.1)
- moved D18 19.9 mm to (191.1, 64.1)
- moved D23 19.9 mm to (248.3, 64.1)
- moved D4 19.9 mm to (38.7, 64.1)
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Routing:
- net SWITCH3-7: track 78.7 -> 98.5 mm, vias 1 -> 3
- net SWITCH2-2: track 171.2 -> 179.7 mm
- net VCC: track 1016.2 -> 1023.2 mm
- net SDA: track 167.0 -> 160.3 mm
- net SWITCH1-5: track 179.7 -> 186.4 mm
- net SWITCH1-8: track 126.7 -> 133.0 mm
- net SWITCH1-2: track 199.7 -> 202.3 mm
- net SWITCH3-1: track 228.9 -> 227.2 mm
- net SWITCH1-6: track 143.0 -> 141.5 mm
- net LED2-4: track 88.2 -> 89.5 mm, vias 1 -> 3
- net SCL: track 168.6 -> 167.3 mm
- net LED1-5: track 139.6 -> 140.8 mm
- net SWITCH2-4: track 141.4 -> 142.5 mm
- net LED2-1: track 100.6 -> 99.4 mm
- net SWITCH1-7: track 302.1 -> 301.5 mm
Other:
- outline, holes or cut-outs redrawn
- board text added: "#4 Screws"
- board text added: "Bridge J1 Jumper"
- board text added: "Display"
- board text added: "Encoder"
- board text added: "MIDI Keyboard V1.0 Apr. 2019 Kyle Lundberg"
- board text added: "Octave+"
- board text added: "Octave-"
- board text added: "Pro Micro"
- board text added: "RESET"
- board text added: "VCC GND SCL SDA"
- board text added: "Velocity"

Commit message: Updated Assembly and Board Tweaks
-Added color to parts in assembly, made renders
-Did final layout adjustments on mainboard. Renamed resistors
Parts:
- R10, R12, R14, R16, R18, R2, R20, R22, R24, R4, R6, R8: value 10k -> (none)
- R25, R27, R29, R31, R33, R35, R37, R39, R41, R43, R45, R47: value (none) -> 10k
- moved R27 137.5 mm to (29.2, 8.89)
- moved R25 135.7 mm to (10.2, 8.89)
- moved R24 135.6 mm to (257.8, 34.3)
- moved R23 128.5 mm to (248.3, 68.6)
- moved R26 128.5 mm to (19.7, 43.8)
- moved R22 124.2 mm to (238.8, 34.3)
- moved R31 120.3 mm to (67.3, 9.53)
- moved R20 117.0 mm to (219.7, 34.3)
- moved R29 117.0 mm to (48.3, 9.53)
- moved R21 114.3 mm to (229.2, 68.6)
- moved R28 114.3 mm to (38.7, 43.8)
- moved R30 110.2 mm to (57.8, 43.8)
- moved R16 104.1 mm to (172.1, 68.6)
- moved R14 104.1 mm to (153.0, 68.6)
- moved R18 98.4 mm to (191.1, 68.6)
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Connections:
- net GND: now also R25.P$2, R27.P$2, R29.P$2, R31.P$2, R33.P$2, R35.P$2, R37.P$2, R39.P$2, R41.P$2, R43.P$2, R45.P$2, R47.P$2; no longer R10.P$2, R12.P$2, R14.P$2, R16.P$2, R18.P$2, R2.P$2, R20.P$2, R22.P$2, R24.P$2, R4.P$2, R6.P$2, R8.P$2
- net LED1-2: now also R2.P$2; no longer R3.P$2
- net LED1-3: now also R3.P$2; no longer R5.P$2
- net LED1-4: now also R4.P$2; no longer R7.P$2
- net LED1-5: now also R5.P$2; no longer R9.P$2
- net LED1-6: now also R6.P$2; no longer R11.P$2
- net LED1-7: now also R7.P$2; no longer R13.P$2
- net LED1-8: now also R8.P$2; no longer R15.P$2
- net LED2-1: now also R9.P$2; no longer R17.P$2
- net LED2-2: now also R10.P$2; no longer R19.P$2
- net LED2-3: now also R11.P$2; no longer R21.P$2
- net LED2-4: now also R12.P$2; no longer R23.P$2
- net LED2-5: now also R13.P$2; no longer R25.P$2
- net LED2-6: now also R14.P$2; no longer R27.P$2
- net LED2-7: now also R15.P$2; no longer R29.P$2
- net LED2-8: now also R16.P$2; no longer R31.P$2
- net LED3-1: now also R17.P$2; no longer R33.P$2
- net LED3-2: now also R18.P$2; no longer R35.P$2
- net LED3-3: now also R19.P$2; no longer R37.P$2
- net LED3-4: now also R20.P$2; no longer R39.P$2
- net LED3-5: now also R21.P$2; no longer R41.P$2
- net LED3-6: now also R22.P$2; no longer R43.P$2
- net LED3-7: now also R23.P$2; no longer R45.P$2
- net LED3-8: now also R24.P$2; no longer R47.P$2
- net N$10: now also R10.P$1; no longer R19.P$1
- net N$11: now also R11.P$1; no longer R21.P$1
- net N$12: now also R12.P$1; no longer R23.P$1
- net N$13: now also R13.P$1; no longer R25.P$1
- net N$14: now also R14.P$1; no longer R27.P$1
- net N$15: now also R15.P$1; no longer R29.P$1
- net N$16: now also R16.P$1; no longer R31.P$1
- net N$17: now also R17.P$1; no longer R33.P$1
- net N$18: now also R18.P$1; no longer R35.P$1
- net N$19: now also R19.P$1; no longer R37.P$1
- net N$2: now also R2.P$1; no longer R3.P$1
- net N$20: now also R20.P$1; no longer R39.P$1
- net N$21: now also R21.P$1; no longer R41.P$1
- net N$22: now also R22.P$1; no longer R43.P$1
- net N$23: now also R23.P$1; no longer R45.P$1
- net N$24: now also R24.P$1; no longer R47.P$1
- net N$3: now also R3.P$1; no longer R5.P$1
- net N$4: now also R4.P$1; no longer R7.P$1
- net N$5: now also R5.P$1; no longer R9.P$1
- net N$6: now also R6.P$1; no longer R11.P$1
- net N$7: now also R7.P$1; no longer R13.P$1
- net N$8: now also R8.P$1; no longer R15.P$1
- net N$9: now also R9.P$1; no longer R17.P$1
- net SWITCH1-1: now also R25.P$1; no longer R2.P$1
- net SWITCH1-2: now also R26.P$1; no longer R4.P$1
- net SWITCH1-3: now also R27.P$1; no longer R6.P$1
- net SWITCH1-4: now also R28.P$1; no longer R8.P$1
- net SWITCH1-5: now also R29.P$1; no longer R10.P$1
- net SWITCH1-6: now also R30.P$1; no longer R12.P$1
- net SWITCH1-7: now also R31.P$1; no longer R14.P$1
- net SWITCH1-8: now also R32.P$1; no longer R16.P$1
- net SWITCH2-1: now also R33.P$1; no longer R18.P$1
- net SWITCH2-2: now also R34.P$1; no longer R20.P$1
- net SWITCH2-3: now also R35.P$1; no longer R22.P$1
- net SWITCH2-4: now also R36.P$1; no longer R24.P$1
- net SWITCH2-5: now also R37.P$1; no longer R26.P$1
- net SWITCH2-6: now also R38.P$1; no longer R28.P$1
- net SWITCH2-7: now also R39.P$1; no longer R30.P$1
- net SWITCH2-8: now also R40.P$1; no longer R32.P$1
- net SWITCH3-1: now also R41.P$1; no longer R34.P$1
- net SWITCH3-2: now also R42.P$1; no longer R36.P$1
- net SWITCH3-3: now also R43.P$1; no longer R38.P$1
- net SWITCH3-4: now also R44.P$1; no longer R40.P$1
- net SWITCH3-5: now also R45.P$1; no longer R42.P$1
- net SWITCH3-6: now also R46.P$1; no longer R44.P$1
- net SWITCH3-7: now also R47.P$1; no longer R46.P$1
Routing:
- net OCTAVE_DOWN: track 227.1 -> 233.0 mm
- net SWITCH3-1: track 227.2 -> 225.7 mm
- net SWITCH1-4: track 165.9 -> 164.4 mm
- net GND: track 343.6 -> 344.8 mm
Other:
- board text added: "#4 SCREWS"
- board text added: "BRIDGE J1 JUMPER"
- board text added: "DISPLAY"
- board text added: "PRO MICRO"
- board text removed: "#4 Screws"
- board text removed: "Bridge J1 Jumper"
- board text removed: "Display"
- board text removed: "Pro Micro"

Commit message: Finished Mainboard and Assembly
-Added mounting holes for display
-Fixed Switch 19 being .05in out of place
Parts:
- moved D17 0.63 mm to (181.6, 29.8)
- moved R17 0.63 mm to (181.6, 34.3)
- moved R41 0.63 mm to (181.6, 9.53)
- moved S17 0.63 mm to (181.6, 19.1)
Routing:
- net LED3-1: track 68.6 -> 69.2 mm
- net SWITCH3-1: track 225.7 -> 226.3 mm
